File: Hardware/Openbook Schematics.sch (EAGLE design)
At the start: 103 parts, among them IC1 BD5229G-TR, IC4 XC6220A331MR-G, J1 FH34SRJ-24S-0.5SH_99_, J2 SAMACSYS_PARTS_USB4110-GF-A, J3 QWIIC_RIGHT_ANGLE, J4 112A-TAAR-R03_ATTEND, Q1 20V/4.2A/52mΩ/1.4W, Q2 20V/4.2A/52mΩ/1.4W, Q3 SI1308EDL-T1-GE3, U1 W25Q512JVEIQ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

Commit message: Fix issues
Parts:
- C3: value 100uF -> 100uF TANT
- EPD_C5: value 1uF/50V -> 0.1uF/50V
Changed lines of the file:
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@@
 <part uuid="2882400001" name="D2" library="DeskAssistant v19 v1" library_urn="urn:adsk.wipprod:fs.file:vf.RKF0zRG-Q6GDTueqQdm8JA" deviceset="ESP32_WROVER_AVX---SD0805S020S1R0_AVX_SD0805S020S1R0_0_0" device="AVX_SD0805S020S1R0_0_0" package3d_urn="urn:adsk.eagle:package:47640134/1" override_locally_modified="yes"/>
 <part uuid="2882400002" name="Q1" library="DeskAssistant v19 v1" library_urn="urn:adsk.wipprod:fs.file:vf.RKF0zRG-Q6GDTueqQdm8JA" deviceset="ESP32_WROVER_SPARKFUN-DISCRETESEMI_MOSFET_PCH" device="-DMG2305UX-7" package3d_urn="urn:adsk.eagle:package:47640135/1" override_locally_modified="yes" value="20V/4.2A/52mΩ/1.4W"/>
-<part uuid="2882400053" name="C3" library="DeskAssistant v19 v1" library_urn="urn:adsk.wipprod:fs.file:vf.RKF0zRG-Q6GDTueqQdm8JA" deviceset="RCL_CPOL-EU" device="CT3528" package3d_urn="urn:adsk.eagle:package:47640137/1" value="100uF"/>
+<part uuid="2882400053" name="C3" library="DeskAssistant v19 v1" library_urn="urn:adsk.wipprod:fs.file:vf.RKF0zRG-Q6GDTueqQdm8JA" deviceset="RCL_CPOL-EU" device="CT3528" package3d_urn="urn:adsk.eagle:package:47640137/1" value="100uF TANT"/>
 <part name="SUPPLY1" library="DeskAssistant v19 v1" library_urn="urn:adsk.wipprod:fs.file:vf.RKF0zRG-Q6GDTueqQdm8JA" deviceset="3V3-CIRCLE" device="" value="3V3"/>
 <part name="C1_BAT2" library="DeskAssistant v19 v1" library_urn="urn:adsk.wipprod:fs.file:vf.RKF0zRG-Q6GDTueqQdm8JA" deviceset="EAGLE-LTSPICE_C" device="C0402" package3d_urn="urn:adsk.eagle:package:47640113/2" value="4.7uF"/>
@@
 <part name="D5" library="DeskAssistant v19 v1" library_urn="urn:adsk.wipprod:fs.file:vf.RKF0zRG-Q6GDTueqQdm8JA" deviceset="MBR0530" device="" package3d_urn="urn:adsk.eagle:package:47640125/3"/>
 <part uuid="2882400025" name="Q3" library="DeskAssistant v19 v1" library_urn="urn:adsk.wipprod:fs.file:vf.RKF0zRG-Q6GDTueqQdm8JA" deviceset="SI1308EDL-T1-GE3" device="" package3d_urn="urn:adsk.eagle:package:47640124/1" override_locally_modified="yes"/>
-<part uuid="2882400051" name="L1" library="DeskAssistant v19 v1" library_urn="urn:adsk.wipprod:fs.file:vf.RKF0zRG-Q6GDTueqQdm8JA" deviceset="744043680" device="IND_4828-WE-TPC_WRE" package3d_urn="urn:adsk.eagle:package:47640123/1" override_locally_modified="yes" value="68uH"/>
+<part uuid="2882400051" name="L1" library="DeskAssistant v19 v1" library_urn="urn:adsk.wipprod:fs.file:vf.RKF0zRG-Q6GDTueqQdm8JA" deviceset="744043680" device="IND_4828-WE-TPC_WRE" package3d_urn="urn:adsk.eagle:package:47640123/2" override_locally_modified="yes" value="68uH"/>
 <part uuid="2882400027" name="U5" library="DeskAssistant v19 v1" library_urn="urn:adsk.wipprod:fs.file:vf.RKF0zRG-Q6GDTueqQdm8JA" deviceset="ESP32_WROVER_SPARKFUN-IC-POWER_MCP73831" device="" package3d_urn="urn:adsk.eagle:package:47640132/1" override_locally_modified="yes"/>
 <part name="GND19" library="DeskAssistant v19 v1" library_urn="urn:adsk.wipprod:fs.file:vf.RKF0zRG-Q6GDTueqQdm8JA" deviceset="GND" device=""/>
@@
 <part name="R_BOOT" library="DeskAssistant v19 v1" library_urn="urn:adsk.wipprod:fs.file:vf.RKF0zRG-Q6GDTueqQdm8JA" deviceset="ESP32_WROVER_EAGLE-LTSPICE_R" device="R0402" package3d_urn="urn:adsk.eagle:package:47640136/3" value="10K"/>
 <part name="R_CHANGE" library="DeskAssistant v19 v1" library_urn="urn:adsk.wipprod:fs.file:vf.RKF0zRG-Q6GDTueqQdm8JA" deviceset="ESP32_WROVER_EAGLE-LTSPICE_R" device="R0402" package3d_urn="urn:adsk.eagle:package:47640136/3" value="10K"/>
-<part uuid="2882400015" name="U4" library="DeskAssistant v19 v1" library_urn="urn:adsk.wipprod:fs.file:vf.RKF0zRG-Q6GDTueqQdm8JA" deviceset="MAX17048G+T10" device="" package3d_urn="urn:adsk.eagle:package:47640119/1" override_locally_modified="yes"/>
+<part uuid="2882400015" name="U4" library="DeskAssistant v19 v1" library_urn="urn:adsk.wipprod:fs.file:vf.RKF0zRG-Q6GDTueqQdm8JA" deviceset="MAX17048G+T10" device="" package3d_urn="urn:adsk.eagle:package:47640119/3" override_locally_modified="yes"/>
 <part name="GND35" library="DeskAssistant v19 v1" library_urn="urn:adsk.wipprod:fs.file:vf.RKF0zRG-Q6GDTueqQdm8JA" deviceset="GND" device=""/>
 <part name="GND36" library="DeskAssistant v19 v1" library_urn="urn:adsk.wipprod:fs.file:vf.RKF0zRG-Q6GDTueqQdm8JA" deviceset="GND" device=""/>
@@
 <part name="EPD_C7" library="DeskAssistant v19 v1" library_urn="urn:adsk.wipprod:fs.file:vf.RKF0zRG-Q6GDTueqQdm8JA" deviceset="EAGLE-LTSPICE_C" device="C0402" package3d_urn="urn:adsk.eagle:package:47640113/2" value="1uF/50V"/>
 <part name="EPD_C6" library="DeskAssistant v19 v1" library_urn="urn:adsk.wipprod:fs.file:vf.RKF0zRG-Q6GDTueqQdm8JA" deviceset="EAGLE-LTSPICE_C" device="C0402" package3d_urn="urn:adsk.eagle:package:47640113/2" value="1uF/50V"/>
-<part name="EPD_C5" library="DeskAssistant v19 v1" library_urn="urn:adsk.wipprod:fs.file:vf.RKF0zRG-Q6GDTueqQdm8JA" deviceset="EAGLE-LTSPICE_C" device="C0402" package3d_urn="urn:adsk.eagle:package:47640113/2" value="1uF/50V"/>
+<part name="EPD_C5" library="DeskAssistant v19 v1" library_urn="urn:adsk.wipprod:fs.file:vf.RKF0zRG-Q6GDTueqQdm8JA" deviceset="EAGLE-LTSPICE_C" device="C0402" package3d_urn="urn:adsk.eagle:package:47640113/2" value="0.1uF/50V"/>
 <part name="EPD_C2" library="DeskAssistant v19 v1" library_urn="urn:adsk.wipprod:fs.file:vf.RKF0zRG-Q6GDTueqQdm8JA" deviceset="EAGLE-LTSPICE_C" device="C0402" package3d_urn="urn:adsk.eagle:package:47640113/2" value="1uF/50V"/>
 <part name="EPD_C1" library="DeskAssistant v19 v1" library_urn="urn:adsk.wipprod:fs.file:vf.RKF0zRG-Q6GDTueqQdm8JA" deviceset="EAGLE-LTSPICE_C" device="C0402" package3d_urn="urn:adsk.eagle:package:47640113/2" value="1uF/50V"/>
@@
 <wire x1="368.3" y1="120.65" x2="377.19" y2="120.65" width="0.1524" layer="91"/>
 <wire x1="377.19" y1="120.65" x2="377.19" y2="123.19" width="0.1524" layer="91"/>
+<pinref part="GND38" gate="1" pin="GND"/>
 <pinref part="U4" gate="G$1" pin="CTG"/>
-<pinref part="GND38" gate="1" pin="GND"/>
 </segment>
 <segment>
 <wire x1="330.2" y1="110.49" x2="330.2" y2="107.95" width="0.1524" layer="91"/>
 <wire x1="330.2" y1="107.95" x2="332.74" y2="107.95" width="0.1524" layer="91"/>
+<pinref part="GND37" gate="1" pin="GND"/>
 <pinref part="U4" gate="G$1" pin="QSTRT"/>
-<pinref part="GND37" gate="1" pin="GND"/>
 </segment>
 <segment>
 <wire x1="368.3" y1="95.25" x2="377.19" y2="95.25" width="0.1524" layer="91"/>
 <wire x1="377.19" y1="95.25" x2="377.19" y2="93.98" width="0.1524" layer="91"/>
+<pinref part="GND36" gate="1" pin="GND"/>
 <pinref part="U4" gate="G$1" pin="GND"/>
-<pinref part="GND36" gate="1" pin="GND"/>
 </segment>
 <segment>
 <wire x1="368.3" y1="113.03" x2="375.92" y2="113.03" width="0.1524" layer="91"/>
+<pinref part="GND35" gate="1" pin="GND"/>
 <pinref part="U4" gate="G$1" pin="EP"/>
-<pinref part="GND35" gate="1" pin="GND"/>
 </segment>
 <segment>
@@
 <junction x="73.66" y="177.8"/>
 <label x="73.66" y="182.88" size="1.016" layer="95" rot="R90" xref="yes"/>
+<pinref part="C7" gate="G$1" pin="1"/>
 <pinref part="L1" gate="A" pin="2"/>
-<pinref part="C7" gate="G$1" pin="1"/>
 </segment>
 <segment>
@@
 <junction x="105.41" y="160.02"/>
 <label x="99.06" y="182.88" size="1.016" layer="95" rot="R90" xref="yes"/>
-<pinref part="L1" gate="A" pin="1"/>
 <pinref part="C4" gate="G$1" pin="2"/>
 <pinref part="D5" gate="G$1" pin="A"/>
-</segment>
-<segment>
+<pinref part="L1" gate="A" pin="1"/>
+</segment>
+<segment>
