File: Hardware/Openbook board.brd (EAGLE design)
At the start: 170.4 x 111.3 mm, 103 parts, among them IC1 BD5229G-TR, IC4 XC6220A331MR-G, J1 FH34SRJ-24S-0.5SH_99_, J2 SAMACSYS_PARTS_USB4110-GF-A, J3 QWIIC_RIGHT_ANGLE, J4 112A-TAAR-R03_ATTEND, Q1 20V/4.2A/52mΩ/1.4W, Q2 20V/4.2A/52mΩ/1.4W, Q3 SI1308EDL-T1-GE3, U1 W25Q512JVEIQ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

Commit message: Fix issues
Parts:
- C3: value 100uF -> 100uF TANT
- EPD_C5: value 1uF/50V -> 0.1uF/50V
- moved TP1 5.95 mm to (6.74, 58.2)
- moved TP10 5.24 mm to (12.8, 10.6)
- moved TP11 4.30 mm to (19.0, 10.4)
- moved TP2 3.90 mm to (12.0, 58.3)
- moved TP9 2.61 mm to (16.5, 58.4)
- moved R1 1.52 mm to (9.52, 17.2)
Routing:
- net GND: track 836.6 -> 806.3 mm, vias 15 -> 47
- net EPD_3V3_C: track 163.6 -> 137.6 mm
- net 3V3: track 453.5 -> 429.6 mm
- net EPD_CS: track 211.2 -> 232.0 mm, vias 7 -> 6
- net USB_D+: track 157.4 -> 139.1 mm
- net N$16: track 13.7 -> 29.6 mm
- net EPD_BUSY: track 131.8 -> 117.0 mm, vias 3 -> 4
- net 32KHZ: track 79.2 -> 65.6 mm, vias 4 -> 3
- net MOSI: track 214.0 -> 202.9 mm, vias 10 -> 8
- net SCK: track 238.2 -> 228.1 mm, vias 8 -> 6
- net SDA: track 195.2 -> 185.2 mm
- net USB_D-: track 132.1 -> 141.3 mm, vias 4 -> 2
- net SCL: track 195.9 -> 187.0 mm
- net EPD_RST: track 150.7 -> 141.9 mm, vias 3 -> 5
- net EPD_DC: track 195.8 -> 187.7 mm, vias 3 -> 5
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